Commit message: Flight once more

File: mantis_description/urdf/arm_link.xacro (robot description, xacro)
@@ -11,5 +11,5 @@
 				<origin xyz="0.091625 0 0" rpy="0 0 0"/>
 				<geometry>
-					<box size="0.18325 0.24 0.041"/>
+					<box size="0.18325 0.024 0.041"/>
 				</geometry>
 			</collision>

File: mantis_description/urdf/mantis.xacro (robot description, xacro)
@@ -4,4 +4,5 @@
 	<xacro:property name="pi" value="3.1415926535897931"/>
 	<!-- Import macros -->
+	<xacro:include filename="$(find mantis_description)/urdf/visual_servo.xacro" />
 	<xacro:include filename="$(find mantis_description)/urdf/frame_battery.xacro" />
 	<xacro:include filename="$(find mantis_description)/urdf/frame_servo.xacro" />
@@ -11,5 +12,5 @@
 	<xacro:include filename="$(find mantis_description)/urdf/arm_joint.xacro" />
 	<xacro:include filename="$(find mantis_description)/urdf/arm_link.xacro" />
-	<xacro:include filename="$(find mantis_description)/urdf/visual_servo.xacro" />
+	<xacro:include filename="$(find mantis_description)/urdf/motor_joint.xacro" />
 	<!-- Import all Gazebo-customization elements, including Gazebo colors -->
 	<xacro:include filename="$(find mantis_description)/urdf/mantis.gazebo" />
@@ -64,3 +65,9 @@
 	<xacro:arm_joint suffix="elbow" parent="link_upperarm" child="link_forearm" xyz="0.18325 0 0" rpy="0 0 0" />
 	<xacro:arm_link suffix="forearm" />
+	<xacro:motor_joint motor_number="1" parent="base_link" xyz="0 -0.275 0.0455" direction="cw" />
+	<xacro:motor_joint motor_number="2" parent="base_link" xyz="0 0.275 0.0475" direction="ccw" />
+	<xacro:motor_joint motor_number="3" parent="base_link" xyz="0.2382 0.1375 0.0455" direction="cw" />
+	<xacro:motor_joint motor_number="4" parent="base_link" xyz="-0.2382 -0.1375 0.0455" direction="ccw" />
+	<xacro:motor_joint motor_number="5" parent="base_link" xyz="0.2382 -0.1375 0.0455" direction="ccw" />
+	<xacro:motor_joint motor_number="6" parent="base_link" xyz="-0.2382 0.1375 0.0455" direction="cw" />
 </robot>

Commit message: RobotModel in rviz is working pretty well now

File: mantis_description/urdf/arm_link.xacro (robot description, xacro)
@@ -19,5 +19,7 @@
 					<mesh filename="package://mantis_description/meshes/FR12-H101.stl" scale="0.001 0.001 0.001"/>
 				</geometry>
-				<material name="black"/>
+				<material name="white">
+					<color rgba="1.0 1.0 1.0 1.0"/>
+				</material>
 			</visual>
 			<visual name="visual_${suffix}_rod">
@@ -26,5 +28,7 @@
 					<mesh filename="package://mantis_description/meshes/rod.stl" scale="0.001 0.001 0.001"/>
 				</geometry>
-				<material name="black"/>
+				<material name="grey">
+					<color rgba="0.2 0.2 0.2 1.0"/>
+				</material>
 			</visual>
 			<xacro:visual_servo suffix="${suffix}" xyz="0.148 0.01425 -0.019" rpy="0 0 ${-pi/2}" />

File: mantis_description/urdf/frame_arm_red.xacro (robot description, xacro)
@@ -1,5 +1,5 @@
 <?xml version="1.0"?>
 <robot xmlns:xacro="http://ros.org/wiki/xacro">
-	<xacro:macro name="frame_arm" params="suffix length radius color xyz rpy">
+	<xacro:macro name="frame_arm_red" params="suffix length radius xyz rpy">
 		<collision name="collision_${suffix}">
 			<origin xyz="${xyz}" rpy="${rpy}"/>
@@ -13,5 +13,7 @@
 				<cylinder radius="${radius}" length="${length}" />
 			</geometry>
-			<material name="${color}"/>
+			<material name="red">
+				<color rgba="1.0 0.0 0.0 1.0"/>
+			</material>
 		</visual>
 	</xacro:macro>

File: mantis_description/urdf/frame_arm_white.xacro (robot description, xacro)
@@ -1,5 +1,5 @@
 <?xml version="1.0"?>
 <robot xmlns:xacro="http://ros.org/wiki/xacro">
-	<xacro:macro name="frame_skid" params="suffix length radius xyz rpy">
+	<xacro:macro name="frame_arm_white" params="suffix length radius xyz rpy">
 		<collision name="collision_${suffix}">
 			<origin xyz="${xyz}" rpy="${rpy}"/>

File: mantis_description/urdf/frame_battery.xacro (robot description, xacro)
@@ -1,5 +1,5 @@
 <?xml version="1.0"?>
 <robot xmlns:xacro="http://ros.org/wiki/xacro">
-	<xacro:macro name="frame_battery" params="suffix size color xyz rpy">
+	<xacro:macro name="frame_battery" params="suffix size xyz rpy">
 		<collision name="collision_${suffix}">
 			<origin xyz="${xyz}" rpy="${rpy}"/>
@@ -13,5 +13,7 @@
 				<box size="${size}"/>
 			</geometry>
-			<material name="${color}"/>
+			<material name="blue">
+				<color rgba="0.0 0.0 0.8 1.0"/>
+			</material>
 		</visual>
 	</xacro:macro>

File: mantis_description/urdf/frame_motor.xacro (robot description, xacro)
@@ -1,5 +1,5 @@
 <?xml version="1.0"?>
 <robot xmlns:xacro="http://ros.org/wiki/xacro">
-	<xacro:macro name="frame_motor" params="suffix length radius color xyz rpy">
+	<xacro:macro name="frame_motor" params="suffix length radius xyz rpy">
 		<collision name="collision_${suffix}">
 			<origin xyz="${xyz}" rpy="${rpy}"/>
@@ -13,5 +13,7 @@
 				<cylinder radius="${radius}" length="${length}" />
 			</geometry>
-			<material name="${color}"/>
+			<material name="grey">
+				<color rgba="0.2 0.2 0.2 1.0"/>
+			</material>
 		</visual>
 	</xacro:macro>

File: mantis_description/urdf/frame_servo.xacro (robot description, xacro)
@@ -1,5 +1,5 @@
 <?xml version="1.0"?>
 <robot xmlns:xacro="http://ros.org/wiki/xacro">
-	<xacro:macro name="frame_servo" params="suffix size color xyz rpy">
+	<xacro:macro name="frame_servo" params="suffix size xyz rpy">
 		<collision name="collision_${suffix}">
 			<origin xyz="${xyz}" rpy="${rpy}"/>

File: mantis_description/urdf/mantis_hex.xacro (robot description, xacro)
@@ -7,5 +7,6 @@
 	<xacro:include filename="$(find mantis_description)/urdf/frame_battery.xacro" />
 	<xacro:include filename="$(find mantis_description)/urdf/frame_servo.xacro" />
-	<xacro:include filename="$(find mantis_description)/urdf/frame_arm.xacro" />
+	<xacro:include filename="$(find mantis_description)/urdf/frame_arm_red.xacro" />
+	<xacro:include filename="$(find mantis_description)/urdf/frame_arm_white.xacro" />
 	<xacro:include filename="$(find mantis_description)/urdf/frame_motor.xacro" />
 	<xacro:include filename="$(find mantis_description)/urdf/frame_skid.xacro" />
@@ -15,6 +16,4 @@
 	<!-- Import all Gazebo-customization elements, including Gazebo colors -->
 	<xacro:include filename="$(find mantis_description)/urdf/mantis.gazebo" />
-	<!-- Import Rviz colors -->
-	<xacro:include filename="$(find mantis_description)/urdf/materials.xacro" />
 	<!-- Used for fixing robot to Gazebo 'base_link' -->
 	<link name="world"/>
@@ -42,26 +41,28 @@
 				<cylinder radius="0.105" length="0.03"/>
 			</geometry>
-			<material name="orange"/>
+			<material name="grey">
+				<color rgba="0.2 0.2 0.2 1.0"/>
+			</material>
 		</visual>
-		<xacro:frame_battery suffix="battery_primary" size="0.052 0.146 0.034" color="blue" xyz="0.0 0.0 0.032" rpy="0.0 0.0 0.0" />
-		<xacro:frame_servo suffix="servo_shoulder" size="0.0285 0.034 0.0465" color="black" xyz="0.01425 0.019 -0.015" rpy="${-pi/2} 0 ${pi}" />
-		<xacro:frame_arm suffix="arm_1" length="0.17" radius="0.015" color="white" xyz="0 -0.19 0" rpy="${pi/2} 0 0" />
-		<xacro:frame_arm suffix="arm_2" length="0.17" radius="0.015" color="white" xyz="0 0.19 0" rpy="${pi/2} 0 0" />
-		<xacro:frame_arm suffix="arm_3" length="0.17" radius="0.015" color="red" xyz="0.165 0.095 0" rpy="${pi/2} 0 ${2*pi/3}" />
-		<xacro:frame_arm suffix="arm_4" length="0.17" radius="0.015" color="white" xyz="-0.165 -0.095 0" rpy="${pi/2} 0 ${2*pi/3}" />
-		<xacro:frame_arm suffix="arm_5" length="0.17" radius="0.015" color="red" xyz="0.165 -0.095 0" rpy="${pi/2} 0 ${pi/3}" />
-		<xacro:frame_arm suffix="arm_6" length="0.17" radius="0.015" color="white" xyz="-0.165 0.095 0" rpy="${pi/2} 0 ${pi/3}" />
-		<xacro:frame_motor suffix="motor_1" length="0.024" radius="0.014" color="grey" xyz="0 -0.275 0.027" rpy="0 0 0" />
-		<xacro:frame_motor suffix="motor_2" length="0.024" radius="0.014" color="grey" xyz="0 0.275 0.027" rpy="0 0 0" />
-		<xacro:frame_motor suffix="motor_3" length="0.024" radius="0.014" color="grey" xyz="0.2382 0.1375 0.027" rpy="0 0 0" />
-		<xacro:frame_motor suffix="motor_4" length="0.024" radius="0.014" color="grey" xyz="-0.2382 -0.1375 0.027" rpy="0 0 0" />
-		<xacro:frame_motor suffix="motor_5" length="0.024" radius="0.014" color="grey" xyz="0.2382 -0.1375 0.027" rpy="0 0 0" />
-		<xacro:frame_motor suffix="motor_6" length="0.024" radius="0.014" color="grey" xyz="-0.2382 0.1375 0.027" rpy="0 0 0" />
-		<xacro:frame_skid suffix="skid_1" length="0.12" radius="0.008" color="white" xyz="0 -0.275 -0.075" rpy="0 0 0" />
-		<xacro:frame_skid suffix="skid_2" length="0.12" radius="0.008" color="white" xyz="0 0.275 -0.075" rpy="0 0 0" />
-		<xacro:frame_skid suffix="skid_3" length="0.12" radius="0.008" color="white" xyz="0.2382 0.1375 -0.075" rpy="0 0 0" />
-		<xacro:frame_skid suffix="skid_4" length="0.12" radius="0.008" color="white" xyz="-0.2382 -0.1375 -0.075" rpy="0 0 0" />
-		<xacro:frame_skid suffix="skid_5" length="0.12" radius="0.008" color="white" xyz="0.2382 -0.1375 -0.075" rpy="0 0 0" />
-		<xacro:frame_skid suffix="skid_6" length="0.12" radius="0.008" color="white" xyz="-0.2382 0.1375 -0.075" rpy="0 0 0" />
+		<xacro:frame_battery suffix="battery_primary" size="0.052 0.146 0.034" xyz="0.0 0.0 0.032" rpy="0.0 0.0 0.0" />
+		<xacro:frame_servo suffix="servo_shoulder" size="0.0285 0.034 0.0465" xyz="0.01425 0.019 -0.015" rpy="${-pi/2} 0 ${pi}" />
+		<xacro:frame_arm_white suffix="arm_1" length="0.17" radius="0.015" xyz="0 -0.19 0" rpy="${pi/2} 0 0" />
+		<xacro:frame_arm_white suffix="arm_2" length="0.17" radius="0.015" xyz="0 0.19 0" rpy="${pi/2} 0 0" />
+		<xacro:frame_arm_red suffix="arm_3" length="0.17" radius="0.015" xyz="0.165 0.095 0" rpy="${pi/2} 0 ${2*pi/3}" />
+		<xacro:frame_arm_white suffix="arm_4" length="0.17" radius="0.015" xyz="-0.165 -0.095 0" rpy="${pi/2} 0 ${2*pi/3}" />
+		<xacro:frame_arm_red suffix="arm_5" length="0.17" radius="0.015" xyz="0.165 -0.095 0" rpy="${pi/2} 0 ${pi/3}" />
+		<xacro:frame_arm_white suffix="arm_6" length="0.17" radius="0.015" xyz="-0.165 0.095 0" rpy="${pi/2} 0 ${pi/3}" />
+		<xacro:frame_motor suffix="motor_1" length="0.024" radius="0.014" xyz="0 -0.275 0.027" rpy="0 0 0" />
+		<xacro:frame_motor suffix="motor_2" length="0.024" radius="0.014" xyz="0 0.275 0.027" rpy="0 0 0" />
+		<xacro:frame_motor suffix="motor_3" length="0.024" radius="0.014" xyz="0.2382 0.1375 0.027" rpy="0 0 0" />
+		<xacro:frame_motor suffix="motor_4" length="0.024" radius="0.014" xyz="-0.2382 -0.1375 0.027" rpy="0 0 0" />
+		<xacro:frame_motor suffix="motor_5" length="0.024" radius="0.014" xyz="0.2382 -0.1375 0.027" rpy="0 0 0" />
+		<xacro:frame_motor suffix="motor_6" length="0.024" radius="0.014" xyz="-0.2382 0.1375 0.027" rpy="0 0 0" />
+		<xacro:frame_skid suffix="skid_1" length="0.12" radius="0.008" xyz="0 -0.275 -0.075" rpy="0 0 0" />
+		<xacro:frame_skid suffix="skid_2" length="0.12" radius="0.008" xyz="0 0.275 -0.075" rpy="0 0 0" />
+		<xacro:frame_skid suffix="skid_3" length="0.12" radius="0.008" xyz="0.2382 0.1375 -0.075" rpy="0 0 0" />
+		<xacro:frame_skid suffix="skid_4" length="0.12" radius="0.008" xyz="-0.2382 -0.1375 -0.075" rpy="0 0 0" />
+		<xacro:frame_skid suffix="skid_5" length="0.12" radius="0.008" xyz="0.2382 -0.1375 -0.075" rpy="0 0 0" />
+		<xacro:frame_skid suffix="skid_6" length="0.12" radius="0.008" xyz="-0.2382 0.1375 -0.075" rpy="0 0 0" />
 	</link>
 	<xacro:arm_joint suffix="shoulder" parent="base_link" child="link_upperarm" xyz="0 0 -0.05025" rpy="${pi/2} ${pi/2} 0" />

File: mantis_description/urdf/mantis_quad.xacro (robot description, xacro)
@@ -7,5 +7,6 @@
 	<xacro:include filename="$(find mantis_description)/urdf/frame_battery.xacro" />
 	<xacro:include filename="$(find mantis_description)/urdf/frame_servo.xacro" />
-	<xacro:include filename="$(find mantis_description)/urdf/frame_arm.xacro" />
+	<xacro:include filename="$(find mantis_description)/urdf/frame_arm_red.xacro" />
+	<xacro:include filename="$(find mantis_description)/urdf/frame_arm_white.xacro" />
 	<xacro:include filename="$(find mantis_description)/urdf/frame_motor.xacro" />
 	<xacro:include filename="$(find mantis_description)/urdf/frame_skid.xacro" />
@@ -15,6 +16,4 @@
 	<!-- Import all Gazebo-customization elements, including Gazebo colors -->
 	<xacro:include filename="$(find mantis_description)/urdf/mantis.gazebo" />
-	<!-- Import Rviz colors -->
-	<xacro:include filename="$(find mantis_description)/urdf/materials.xacro" />
 	<!-- Used for fixing robot to Gazebo 'base_link' -->
 	<link name="world"/>
@@ -42,20 +41,22 @@
 				<cylinder radius="0.075" length="0.03"/>
 			</geometry>
-			<material name="orange"/>
+			<material name="grey">
+				<color rgba="0.2 0.2 0.2 1.0"/>
+			</material>
 		</visual>
-		<xacro:frame_battery suffix="battery_primary" size="0.052 0.146 0.034" color="blue" xyz="0.0 0.0 0.032" rpy="0.0 0.0 0.0" />
-		<xacro:frame_servo suffix="servo_shoulder" size="0.0285 0.034 0.0465" color="black" xyz="0.01425 0.019 -0.015" rpy="${-pi/2} 0 ${pi}" />
-		<xacro:frame_arm suffix="arm_1" length="0.15" radius="0.015" color="white" xyz="0.1061 -0.1061 0" rpy="${pi/2} 0 ${pi/4}" />
-		<xacro:frame_arm suffix="arm_2" length="0.15" radius="0.015" color="white" xyz="-0.1061 0.1061 0" rpy="${pi/2} 0 ${pi/4}" />
-		<xacro:frame_arm suffix="arm_3" length="0.15" radius="0.015" color="red" xyz="0.1061 0.1061 0" rpy="${pi/2} 0 ${-pi/4}" />
-		<xacro:frame_arm suffix="arm_4" length="0.15" radius="0.015" color="white" xyz="-0.1061 -0.1061 0" rpy="${pi/2} 0 ${-pi/4}" />
-		<xacro:frame_motor suffix="motor_1" length="0.024" radius="0.014" color="grey" xyz="0.1591 -0.1591 0.027" rpy="0 0 0" />
-		<xacro:frame_motor suffix="motor_2" length="0.024" radius="0.014" color="grey" xyz="-0.1591 0.1591 0.027" rpy="0 0 0" />
-		<xacro:frame_motor suffix="motor_3" length="0.024" radius="0.014" color="grey" xyz="0.1591 0.1591 0.027" rpy="0 0 0" />
-		<xacro:frame_motor suffix="motor_4" length="0.024" radius="0.014" color="grey" xyz="-0.1591 -0.1591 0.027" rpy="0 0 0" />
-		<xacro:frame_skid suffix="skid_1" length="0.12" radius="0.008" color="white" xyz="0.1591 -0.1591 -0.075" rpy="0 0 0" />
-		<xacro:frame_skid suffix="skid_2" length="0.12" radius="0.008" color="white" xyz="-0.1591 0.1591 -0.075" rpy="0 0 0" />
-		<xacro:frame_skid suffix="skid_3" length="0.12" radius="0.008" color="white" xyz="0.1591 0.1591 -0.075" rpy="0 0 0" />
-		<xacro:frame_skid suffix="skid_4" length="0.12" radius="0.008" color="white" xyz="-0.1591 -0.1591 -0.075" rpy="0 0 0" />
+		<xacro:frame_battery suffix="battery_primary" size="0.052 0.146 0.034" xyz="0.0 0.0 0.032" rpy="0.0 0.0 0.0" />
+		<xacro:frame_servo suffix="servo_shoulder" size="0.0285 0.034 0.0465" xyz="0.01425 0.019 -0.015" rpy="${-pi/2} 0 ${pi}" />
+		<xacro:frame_arm_red suffix="arm_1" length="0.15" radius="0.015" xyz="0.1061 -0.1061 0" rpy="${pi/2} 0 ${pi/4}" />
+		<xacro:frame_arm_white suffix="arm_2" length="0.15" radius="0.015" xyz="-0.1061 0.1061 0" rpy="${pi/2} 0 ${pi/4}" />
+		<xacro:frame_arm_red suffix="arm_3" length="0.15" radius="0.015" xyz="0.1061 0.1061 0" rpy="${pi/2} 0 ${-pi/4}" />
+		<xacro:frame_arm_white suffix="arm_4" length="0.15" radius="0.015" xyz="-0.1061 -0.1061 0" rpy="${pi/2} 0 ${-pi/4}" />
+		<xacro:frame_motor suffix="motor_1" length="0.024" radius="0.014" xyz="0.1591 -0.1591 0.027" rpy="0 0 0" />
+		<xacro:frame_motor suffix="motor_2" length="0.024" radius="0.014" xyz="-0.1591 0.1591 0.027" rpy="0 0 0" />
+		<xacro:frame_motor suffix="motor_3" length="0.024" radius="0.014" xyz="0.1591 0.1591 0.027" rpy="0 0 0" />
+		<xacro:frame_motor suffix="motor_4" length="0.024" radius="0.014" xyz="-0.1591 -0.1591 0.027" rpy="0 0 0" />
+		<xacro:frame_skid suffix="skid_1" length="0.12" radius="0.008" xyz="0.1591 -0.1591 -0.075" rpy="0 0 0" />
+		<xacro:frame_skid suffix="skid_2" length="0.12" radius="0.008" xyz="-0.1591 0.1591 -0.075" rpy="0 0 0" />
+		<xacro:frame_skid suffix="skid_3" length="0.12" radius="0.008" xyz="0.1591 0.1591 -0.075" rpy="0 0 0" />
+		<xacro:frame_skid suffix="skid_4" length="0.12" radius="0.008" xyz="-0.1591 -0.1591 -0.075" rpy="0 0 0" />
 	</link>
 	<xacro:arm_joint suffix="shoulder" parent="base_link" child="link_upperarm" xyz="0 0 -0.05025" rpy="${pi/2} ${pi/2} 0" />

File: mantis_description/urdf/visual_servo.xacro (robot description, xacro)
@@ -7,5 +7,7 @@
 				<mesh filename="package://mantis_description/meshes/X-430_IDLE.stl" scale="0.001 0.001 0.001"/>
 			</geometry>
-			<material name="black"/>
+			<material name="dark_grey">
+				<color rgba="0.1 0.1 0.1 1.0"/>
+			</material>
 		</visual>
 	</xacro:macro>
