Commit message: Making xacro a bit more modular

File: mantis_description/urdf/arm_link.xacro (robot description, xacro)
@@ -1,4 +1,5 @@
 <?xml version="1.0"?>
 <robot xmlns:xacro="http://ros.org/wiki/xacro">
+	<xacro:include filename="$(find mantis_description)/urdf/visual_servo.xacro" />
 	<xacro:macro name="arm_link" params="suffix">
 		<link name="link_${suffix}">

File: mantis_description/urdf/frame_servo.xacro (robot description, xacro)
@@ -1,4 +1,5 @@
 <?xml version="1.0"?>
 <robot xmlns:xacro="http://ros.org/wiki/xacro">
+	<xacro:include filename="$(find mantis_description)/urdf/visual_servo.xacro" />
 	<xacro:macro name="frame_servo" params="suffix size xyz rpy">
 		<collision name="collision_${suffix}">

File: mantis_description/urdf/mantis_hex.xacro (robot description, xacro)
@@ -4,14 +4,7 @@
 	<xacro:property name="pi" value="3.1415926535897931"/>
 	<!-- Import macros -->
-	<xacro:include filename="$(find mantis_description)/urdf/visual_servo.xacro" />
-	<xacro:include filename="$(find mantis_description)/urdf/frame_battery.xacro" />
-	<xacro:include filename="$(find mantis_description)/urdf/frame_servo.xacro" />
-	<xacro:include filename="$(find mantis_description)/urdf/frame_arm_red.xacro" />
-	<xacro:include filename="$(find mantis_description)/urdf/frame_arm_white.xacro" />
-	<xacro:include filename="$(find mantis_description)/urdf/frame_motor.xacro" />
-	<xacro:include filename="$(find mantis_description)/urdf/frame_skid.xacro" />
+	<xacro:include filename="$(find mantis_description)/urdf/base_hex.xacro" />
 	<xacro:include filename="$(find mantis_description)/urdf/arm_joint.xacro" />
 	<xacro:include filename="$(find mantis_description)/urdf/arm_link.xacro" />
-	<xacro:include filename="$(find mantis_description)/urdf/motor_joint.xacro" />
 	<!-- Import all Gazebo-customization elements, including Gazebo colors -->
 	<xacro:include filename="$(find mantis_description)/urdf/mantis.gazebo" />
@@ -22,82 +15,8 @@
 		<child link="base_link"/>
 	</joint>
-	<!-- Base Link -->
-	<link name="base_link">
-		<inertial>
-			<!-- Old estimate
-			<mass value="1.5480" />
-			<inertia ixx="0.015198135489664" iyy="0.014353211169664" izz="0.027767959346667" ixy="0.0" ixz="0.0" iyz="0.0" />
-			-->
-			<mass value="1.80497" />
-			<inertia ixx="0.02961" iyy="0.02933" izz="0.05342" ixy="0.0" ixz="0.00004" iyz="0.0" />
-		</inertial>
-		<collision name='collision_base_link'>
-			<geometry>
-				<cylinder radius="0.105" length="0.03"/>
-			</geometry>
-		</collision>
-		<visual name='visual_base_link'>
-			<geometry>
-				<cylinder radius="0.105" length="0.03"/>
-			</geometry>
-			<material name="grey">
-				<color rgba="0.2 0.2 0.2 1.0"/>
-			</material>
-		</visual>
-		<xacro:frame_battery suffix="battery_primary" size="0.052 0.146 0.034" xyz="0.0 0.0 0.032" rpy="0.0 0.0 0.0" />
-		<xacro:frame_servo suffix="servo_shoulder" size="0.0285 0.034 0.0465" xyz="0.01425 0.019 -0.015" rpy="${-pi/2} 0 ${pi}" />
-		<xacro:frame_arm_white suffix="arm_1" length="0.17" radius="0.015" xyz="0 -0.19 0" rpy="${pi/2} 0 0" />
-		<xacro:frame_arm_white suffix="arm_2" length="0.17" radius="0.015" xyz="0 0.19 0" rpy="${pi/2} 0 0" />
-		<xacro:frame_arm_red suffix="arm_3" length="0.17" radius="0.015" xyz="0.165 0.095 0" rpy="${pi/2} 0 ${2*pi/3}" />
-		<xacro:frame_arm_white suffix="arm_4" length="0.17" radius="0.015" xyz="-0.165 -0.095 0" rpy="${pi/2} 0 ${2*pi/3}" />
-		<xacro:frame_arm_red suffix="arm_5" length="0.17" radius="0.015" xyz="0.165 -0.095 0" rpy="${pi/2} 0 ${pi/3}" />
-		<xacro:frame_arm_white suffix="arm_6" length="0.17" radius="0.015" xyz="-0.165 0.095 0" rpy="${pi/2} 0 ${pi/3}" />
-		<xacro:frame_motor suffix="motor_1" length="0.024" radius="0.014" xyz="0 -0.275 0.027" rpy="0 0 0" />
-		<xacro:frame_motor suffix="motor_2" length="0.024" radius="0.014" xyz="0 0.275 0.027" rpy="0 0 0" />
-		<xacro:frame_motor suffix="motor_3" length="0.024" radius="0.014" xyz="0.2382 0.1375 0.027" rpy="0 0 0" />
-		<xacro:frame_motor suffix="motor_4" length="0.024" radius="0.014" xyz="-0.2382 -0.1375 0.027" rpy="0 0 0" />
-		<xacro:frame_motor suffix="motor_5" length="0.024" radius="0.014" xyz="0.2382 -0.1375 0.027" rpy="0 0 0" />
-		<xacro:frame_motor suffix="motor_6" length="0.024" radius="0.014" xyz="-0.2382 0.1375 0.027" rpy="0 0 0" />
-		<xacro:frame_skid suffix="skid_1" length="0.12" radius="0.008" xyz="0 -0.275 -0.075" rpy="0 0 0" />
-		<xacro:frame_skid suffix="skid_2" length="0.12" radius="0.008" xyz="0 0.275 -0.075" rpy="0 0 0" />
-		<xacro:frame_skid suffix="skid_3" length="0.12" radius="0.008" xyz="0.2382 0.1375 -0.075" rpy="0 0 0" />
-		<xacro:frame_skid suffix="skid_4" length="0.12" radius="0.008" xyz="-0.2382 -0.1375 -0.075" rpy="0 0 0" />
-		<xacro:frame_skid suffix="skid_5" length="0.12" radius="0.008" xyz="0.2382 -0.1375 -0.075" rpy="0 0 0" />
-		<xacro:frame_skid suffix="skid_6" length="0.12" radius="0.008" xyz="-0.2382 0.1375 -0.075" rpy="0 0 0" />
-	</link>
+	<xacro:base_hex arm_length="0.17" base_radius="0.105" mass="1.80497" ixx="0.02961" iyy="0.02933" izz="0.05342" ixy="0.0" ixz="0.00004" iyz="0.0" />
 	<xacro:arm_joint suffix="shoulder" parent="base_link" child="link_upperarm" xyz="0 0 -0.05025" rpy="${pi/2} ${pi/2} 0" />
 	<xacro:arm_link suffix="upperarm" />
 	<xacro:arm_joint suffix="elbow" parent="link_upperarm" child="link_forearm" xyz="0.18325 0 0" rpy="0 0 0" />
 	<xacro:arm_link suffix="forearm" />
-	<!--
-	<joint name="joint_wrist" type="fixed">
-		<parent link="link_forearm"/>
-		<child link="link_end_effector"/>
-		<origin xyz="0.18325 0 0" rpy="0 0 0"/>
-	</joint>
-	<link name="link_end_effector">
-		<inertial name='inertial_end_effector'>>
-			<origin xyz="0.025 0 0" rpy="0 0 0"/>
-			<mass value="0.001" />
-			<inertia ixx="1.0e-07" iyy="1.0e-07" izz="1.0e-07" ixy="0.0" ixz="0.0" iyz="0.0" />
-		</inertial>
-		<collision name='collision_end_effector'>
-			<geometry>
-				<box size="0.05 0.05 0.05"/>
-			</geometry>
-		</collision>
-		<visual name="visual_end_effector">
-			<geometry>
-				<box size="0.05 0.05 0.05"/>
-			</geometry>
-			<material name="black"/>
-		</visual>
-	</link>
-	-->
-	<xacro:motor_joint motor_number="1" parent="base_link" xyz="0 -0.275 0.0455" direction="cw" />
-	<xacro:motor_joint motor_number="2" parent="base_link" xyz="0 0.275 0.0475" direction="ccw" />
-	<xacro:motor_joint motor_number="3" parent="base_link" xyz="0.2382 0.1375 0.0455" direction="cw" />
-	<xacro:motor_joint motor_number="4" parent="base_link" xyz="-0.2382 -0.1375 0.0455" direction="ccw" />
-	<xacro:motor_joint motor_number="5" parent="base_link" xyz="0.2382 -0.1375 0.0455" direction="ccw" />
-	<xacro:motor_joint motor_number="6" parent="base_link" xyz="-0.2382 0.1375 0.0455" direction="cw" />
 </robot>

File: mantis_description/urdf/mantis_quad.xacro (robot description, xacro)
@@ -4,14 +4,7 @@
 	<xacro:property name="pi" value="3.1415926535897931"/>
 	<!-- Import macros -->
-	<xacro:include filename="$(find mantis_description)/urdf/visual_servo.xacro" />
-	<xacro:include filename="$(find mantis_description)/urdf/frame_battery.xacro" />
-	<xacro:include filename="$(find mantis_description)/urdf/frame_servo.xacro" />
-	<xacro:include filename="$(find mantis_description)/urdf/frame_arm_red.xacro" />
-	<xacro:include filename="$(find mantis_description)/urdf/frame_arm_white.xacro" />
-	<xacro:include filename="$(find mantis_description)/urdf/frame_motor.xacro" />
-	<xacro:include filename="$(find mantis_description)/urdf/frame_skid.xacro" />
+	<xacro:include filename="$(find mantis_description)/urdf/base_quad.xacro" />
 	<xacro:include filename="$(find mantis_description)/urdf/arm_joint.xacro" />
 	<xacro:include filename="$(find mantis_description)/urdf/arm_link.xacro" />
-	<xacro:include filename="$(find mantis_description)/urdf/motor_joint.xacro" />
 	<!-- Import all Gazebo-customization elements, including Gazebo colors -->
 	<xacro:include filename="$(find mantis_description)/urdf/mantis.gazebo" />
@@ -22,74 +15,8 @@
 		<child link="base_link"/>
 	</joint>
-	<!-- Base Link -->
-	<link name="base_link">
-		<inertial>
-			<!-- Old estimate
-			<mass value="1.5480" />
-			<inertia ixx="0.015198135489664" iyy="0.014353211169664" izz="0.027767959346667" ixy="0.0" ixz="0.0" iyz="0.0" />
-			-->
-			<mass value="1.80497" />
-			<inertia ixx="0.02961" iyy="0.02933" izz="0.05342" ixy="0.0" ixz="0.00004" iyz="0.0" />
-		</inertial>
-		<collision name='collision_base_link'>
-			<geometry>
-				<cylinder radius="0.075" length="0.03"/>
-			</geometry>
-		</collision>
-		<visual name='visual_base_link'>
-			<geometry>
-				<cylinder radius="0.075" length="0.03"/>
-			</geometry>
-			<material name="grey">
-				<color rgba="0.2 0.2 0.2 1.0"/>
-			</material>
-		</visual>
-		<xacro:frame_battery suffix="battery_primary" size="0.052 0.146 0.034" xyz="0.0 0.0 0.032" rpy="0.0 0.0 0.0" />
-		<xacro:frame_servo suffix="servo_shoulder" size="0.0285 0.034 0.0465" xyz="0.01425 0.019 -0.015" rpy="${-pi/2} 0 ${pi}" />
-		<xacro:frame_arm_red suffix="arm_1" length="0.15" radius="0.015" xyz="0.1061 -0.1061 0" rpy="${pi/2} 0 ${pi/4}" />
-		<xacro:frame_arm_white suffix="arm_2" length="0.15" radius="0.015" xyz="-0.1061 0.1061 0" rpy="${pi/2} 0 ${pi/4}" />
-		<xacro:frame_arm_red suffix="arm_3" length="0.15" radius="0.015" xyz="0.1061 0.1061 0" rpy="${pi/2} 0 ${-pi/4}" />
-		<xacro:frame_arm_white suffix="arm_4" length="0.15" radius="0.015" xyz="-0.1061 -0.1061 0" rpy="${pi/2} 0 ${-pi/4}" />
-		<xacro:frame_motor suffix="motor_1" length="0.024" radius="0.014" xyz="0.1591 -0.1591 0.027" rpy="0 0 0" />
-		<xacro:frame_motor suffix="motor_2" length="0.024" radius="0.014" xyz="-0.1591 0.1591 0.027" rpy="0 0 0" />
-		<xacro:frame_motor suffix="motor_3" length="0.024" radius="0.014" xyz="0.1591 0.1591 0.027" rpy="0 0 0" />
-		<xacro:frame_motor suffix="motor_4" length="0.024" radius="0.014" xyz="-0.1591 -0.1591 0.027" rpy="0 0 0" />
-		<xacro:frame_skid suffix="skid_1" length="0.12" radius="0.008" xyz="0.1591 -0.1591 -0.075" rpy="0 0 0" />
-		<xacro:frame_skid suffix="skid_2" length="0.12" radius="0.008" xyz="-0.1591 0.1591 -0.075" rpy="0 0 0" />
-		<xacro:frame_skid suffix="skid_3" length="0.12" radius="0.008" xyz="0.1591 0.1591 -0.075" rpy="0 0 0" />
-		<xacro:frame_skid suffix="skid_4" length="0.12" radius="0.008" xyz="-0.1591 -0.1591 -0.075" rpy="0 0 0" />
-	</link>
+	<xacro:base_quad arm_length="0.15" base_radius="0.075" mass="1.80497" ixx="0.02961" iyy="0.02933" izz="0.05342" ixy="0.0" ixz="0.00004" iyz="0.0" />
 	<xacro:arm_joint suffix="shoulder" parent="base_link" child="link_upperarm" xyz="0 0 -0.05025" rpy="${pi/2} ${pi/2} 0" />
 	<xacro:arm_link suffix="upperarm" />
 	<xacro:arm_joint suffix="elbow" parent="link_upperarm" child="link_forearm" xyz="0.18325 0 0" rpy="0 0 0" />
 	<xacro:arm_link suffix="forearm" />
-	<!--
-	<joint name="joint_wrist" type="fixed">
-		<parent link="link_forearm"/>
-		<child link="link_end_effector"/>
-		<origin xyz="0.18325 0 0" rpy="0 0 0"/>
-	</joint>
-	<link name="link_end_effector">
-		<inertial name='inertial_end_effector'>>
-			<origin xyz="0.025 0 0" rpy="0 0 0"/>
-			<mass value="0.001" />
-			<inertia ixx="1.0e-07" iyy="1.0e-07" izz="1.0e-07" ixy="0.0" ixz="0.0" iyz="0.0" />
-		</inertial>
-		<collision name='collision_end_effector'>
-			<geometry>
-				<box size="0.05 0.05 0.05"/>
-			</geometry>
-		</collision>
-		<visual name="visual_end_effector">
-			<geometry>
-				<box size="0.05 0.05 0.05"/>
-			</geometry>
-			<material name="black"/>
-		</visual>
-	</link>
-	-->
-	<xacro:motor_joint motor_number="1" parent="base_link" xyz="0.1591 -0.1591 0.0455" direction="ccw" />
-	<xacro:motor_joint motor_number="2" parent="base_link" xyz="-0.1591 0.1591 0.0475" direction="ccw" />
-	<xacro:motor_joint motor_number="3" parent="base_link" xyz="0.1591 0.1591 0.0455" direction="cw" />
-	<xacro:motor_joint motor_number="4" parent="base_link" xyz="-0.1591 -0.1591 0.0455" direction="cw" />
 </robot>
