Commit message: Started slung load example

File: mantis_description/urdf/base_hex_single_servo.xacro (robot description, xacro)
@@ -8,5 +8,5 @@
 	<xacro:include filename="$(find mantis_description)/urdf/frame_skid.xacro" />
 	<xacro:include filename="$(find mantis_description)/urdf/motor_joint.xacro" />
-	<xacro:macro name="base_hex" params="arm_length base_radius mass ixx iyy izz ixy ixz iyz">
+	<xacro:macro name="base_hex_single_servo" params="arm_length base_radius mass ixx iyy izz ixy ixz iyz">
 		<!-- Base Link -->
 		<link name="base_link">

File: mantis_description/urdf/base_quad_wire.xacro (robot description, xacro)
@@ -2,5 +2,4 @@
 <robot xmlns:xacro="http://ros.org/wiki/xacro">
 	<xacro:include filename="$(find mantis_description)/urdf/frame_battery.xacro" />
-	<xacro:include filename="$(find mantis_description)/urdf/frame_servo.xacro" />
 	<xacro:include filename="$(find mantis_description)/urdf/frame_arm_red.xacro" />
 	<xacro:include filename="$(find mantis_description)/urdf/frame_arm_white.xacro" />
@@ -8,5 +7,5 @@
 	<xacro:include filename="$(find mantis_description)/urdf/frame_skid.xacro" />
 	<xacro:include filename="$(find mantis_description)/urdf/motor_joint.xacro" />
-	<xacro:macro name="base_quad" params="arm_length base_radius mass ixx iyy izz ixy ixz iyz">
+	<xacro:macro name="base_quad_wire" params="arm_length base_radius mass ixx iyy izz ixy ixz iyz">
 		<!-- Base Link -->
 		<link name="base_link">
@@ -33,5 +32,4 @@
 			</visual>
 			<xacro:frame_battery suffix="battery_primary" size="0.052 0.146 0.034" xyz="0.0 0.0 0.032" rpy="0.0 0.0 0.0" />
-			<xacro:frame_servo suffix="servo_shoulder" size="0.0285 0.034 0.0465" xyz="0.01425 0.019 -0.015" rpy="${-pi/2} 0 ${pi}" />
 			<xacro:frame_arm_red suffix="arm_1" length="${arm_length}" radius="0.015" xyz="0.1061 -0.1061 0" rpy="${pi/2} 0 ${pi/4}" />
 			<xacro:frame_arm_white suffix="arm_2" length="${arm_length}" radius="0.015" xyz="-0.1061 0.1061 0" rpy="${pi/2} 0 ${pi/4}" />

File: mantis_description/urdf/mantis_hex.xacro (robot description, xacro)
@@ -4,5 +4,5 @@
 	<xacro:property name="pi" value="3.1415926535897931"/>
 	<!-- Import macros -->
-	<xacro:include filename="$(find mantis_description)/urdf/base_hex.xacro" />
+	<xacro:include filename="$(find mantis_description)/urdf/base_hex_single_servo.xacro" />
 	<xacro:include filename="$(find mantis_description)/urdf/arm_joint.xacro" />
 	<xacro:include filename="$(find mantis_description)/urdf/arm_link.xacro" />
@@ -15,5 +15,5 @@
 		<child link="base_link"/>
 	</joint>
-	<xacro:base_hex arm_length="0.17" base_radius="0.105" mass="1.80497" ixx="0.02961" iyy="0.02933" izz="0.05342" ixy="0.0" ixz="0.00004" iyz="0.0" />
+	<xacro:base_hex_single_servo arm_length="0.17" base_radius="0.105" mass="1.80497" ixx="0.02961" iyy="0.02933" izz="0.05342" ixy="0.0" ixz="0.00004" iyz="0.0" />
 	<xacro:arm_joint suffix="shoulder" parent="base_link" child="link_upperarm" xyz="0 0 -0.05025" rpy="${pi/2} ${pi/2} 0" />
 	<xacro:arm_link suffix="upperarm" />

File: mantis_description/urdf/mantis_quad.xacro (robot description, xacro)
@@ -4,5 +4,5 @@
 	<xacro:property name="pi" value="3.1415926535897931"/>
 	<!-- Import macros -->
-	<xacro:include filename="$(find mantis_description)/urdf/base_quad.xacro" />
+	<xacro:include filename="$(find mantis_description)/urdf/base_quad_single_servo.xacro" />
 	<xacro:include filename="$(find mantis_description)/urdf/arm_joint.xacro" />
 	<xacro:include filename="$(find mantis_description)/urdf/arm_link.xacro" />
@@ -15,5 +15,5 @@
 		<child link="base_link"/>
 	</joint>
-	<xacro:base_quad arm_length="0.15" base_radius="0.075" mass="1.80497" ixx="0.02961" iyy="0.02933" izz="0.05342" ixy="0.0" ixz="0.00004" iyz="0.0" />
+	<xacro:base_quad_single_servo arm_length="0.15" base_radius="0.075" mass="1.80497" ixx="0.02961" iyy="0.02933" izz="0.05342" ixy="0.0" ixz="0.00004" iyz="0.0" />
 	<xacro:arm_joint suffix="shoulder" parent="base_link" child="link_upperarm" xyz="0 0 -0.05025" rpy="${pi/2} ${pi/2} 0" />
 	<xacro:arm_link suffix="upperarm" />
